File: OpenAmiga500FastRamExpansion.sch (KiCad schematic (older format))
At the start: 35 parts, among them J1 68000_SOCKET, P1 JTAG_CONNECTOR, P99 OSHW_LOGO, U1 68000D, U2 74LS157, U3 74LS157, U4 ATF1502AS-10JU44, U5 HYB5118160BSJ, U6 HYB5118160BSJ, U7 HYB5118160BSJ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

Commit message: Autoconfig improvements * Add CFGIN * Add hardware to hide autoconfig cycles until configured   - Config before others   - No need for cfgout   - No need for cfgin if you want it to be the first dev configured
As of yet untested, waiting on parts and need to adapt code :)
Parts:
- added C20, C21, C22: 100n, Capacitor_SMD:C_0805_2012Metric_Pad1.18x1.45mm_HandSolder, symbol Device:C
- added J2: ~cfgin, Connector_PinHeader_2.54mm:PinHeader_1x01_P2.54mm_Horizontal, symbol Connector:Conn_01x01_Male
- added R5, R6: 4k7, Resistor_SMD:R_0805_2012Metric_Pad1.20x1.40mm_HandSolder, symbol Device:R_Small
- added R7: 10k, Resistor_SMD:R_0805_2012Metric_Pad1.20x1.40mm_HandSolder, symbol Device:R
- added U10: 74AHCT257, Package_SO:SOIC-16_3.9x9.9mm_P1.27mm, symbol 74xx:74LS257
- added U11: 74AHC00, Package_SO:SOIC-14_3.9x8.7mm_P1.27mm, symbol 74xx:74HC00
- added U9: 74LS157, Package_SO:SOIC-16_3.9x9.9mm_P1.27mm, symbol 74xx:74LS157
- P1: symbol conn:CONN_5X2 -> OpenAmiga500FastRamExpansion-rescue:CONN_5X2-conn
- P99: symbol conn:CONN_1 -> OpenAmiga500FastRamExpansion-rescue:CONN_1-conn
Connections:
- net labels added: DMA, lds, uds, ~blds, ~buds, ~cfgin, ~cloak, ~cpulds, ~cpuuds
- net labels removed: ~lds, ~uds
- wire segments 500 -> 566
- no-connect marks 24 -> 29
Other:
- note added: "Cloaking circuitry\n"
- note added: "DMA hacks"
- note added: "During DMA some other bus master will drive UDS/LDS\nSo we need to tri-state the cloak's outputs.\nThe CPLD needs to receive the bus masters UDS/LDS\nThese NAND gates provide that whether the CPU or something else is bus master"
- note added: "Hide autoconfig cycles from rest of system during our turn\nPrevents conflicts without needing cfgin/out"
- moved on the sheet: C1, C2, C3, C4, C5, C6, C7, LD1, R1, R2, R3, R4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

Commit message: Isolate /AS too
Connections:
- net labels added: as, ~bas, ~bdtack, ~cpuas, ~cpudtack
- net labels removed: ~as, ~dtack
- wire segments 566 -> 564
- no-connect marks 29 -> 26
Other:
- note added: "During DMA some other bus master will drive UDS/LDS/AS\nSo we need to tri-state the cloak's outputs.\nThe CPLD needs to receive the bus masters UDS/LDS/AS\nThese NAND gates provide that whether the CPU or something else is bus master"
- note removed: "During DMA some other bus master will drive UDS/LDS\nSo we need to tri-state the cloak's outputs.\nThe CPLD needs to receive the bus masters UDS/LDS\nThese NAND gates provide that whether the CPU or something else is bus master"
- moved on the sheet: C21, R5, R6, U10

Commit message: Add V2 Firmware, update documentation
Parts:
- added J3: 4MB, Connector_PinHeader_2.54mm:PinHeader_1x02_P2.54mm_Horizontal, symbol Connector:Conn_01x02_Male
- added R8, R9: 4k7, Resistor_SMD:R_0805_2012Metric_Pad1.20x1.40mm_HandSolder, symbol Device:R
- J2: value ~cfgin -> cfgin
- R7: value 10k -> 4k7
- U10: value 74AHCT257 -> 74ALS257
- U11: value 74AHC00 -> 74AHCT00
- U2, U3, U9: value 74LS157 -> 74AHCT157
Connections:
- net labels added: cfg
- net labels removed: ~cfgin
- wire segments 564 -> 568
- no-connect marks 26 -> 25
Other:
- note added: "NOTE!\nDO NOT substitute for a different logic family\nU10's Timing and drive characteristics are critical"
- moved on the sheet: C2, C20, C21, C3, J2, R5, R6, R7, U10, U2, U3, U4

Commit message: Fixup schematic + documentation
Parts:
- U4: value ATF1502AS-10JU44 -> ATF1504AS-10JU44
Changed lines of the file:
@@
 P 5410 10430
 F 0 "U4" H 5350 10460 50  0000 L CNN
-F 1 "ATF1502AS-10JU44" H 5120 10370 50  0000 L CNN
+F 1 "ATF1504AS-10JU44" H 5120 10370 50  0000 L CNN
 F 2 "OpenAmiga500FastRamExpansion:PLCC-44_THT-Socket" H 5410 10430 50  0001 C CNN
 F 3 "DOCUMENTATION" H 5410 10430 50  0001 C CNN
@@
 Wire Wire Line
 	11900 9400 12440 9400
-Wire Bus Line
-	8370 3300 8370 7610
-Wire Bus Line
-	11790 3300 11790 7610
-Wire Bus Line
-	14260 3300 14260 7610
-Wire Bus Line
-	3650 3670 3650 5170
-Wire Bus Line
-	7180 3670 7180 5170
-Wire Bus Line
-	10840 3300 10840 7610
-Wire Bus Line
-	11230 970  11230 5820
-Wire Bus Line
-	8130 970  8130 5620
-Wire Bus Line
-	7180 1260 7180 3470
-Wire Bus Line
-	3650 1260 3650 3470
-Wire Bus Line
-	14650 970  14650 5820
-Wire Bus Line
-	11550 970  11550 5620
 $Comp
 L 74xx:74LS157 U9
@@
 	1    0    0    -1
 $EndComp
+Wire Bus Line
+	8370 3300 8370 7610
+Wire Bus Line
+	11790 3300 11790 7610
+Wire Bus Line
+	14260 3300 14260 7610
+Wire Bus Line
+	3650 3670 3650 5170
+Wire Bus Line
+	7180 3670 7180 5170
+Wire Bus Line
+	10840 3300 10840 7610
+Wire Bus Line
+	11230 970  11230 5820
+Wire Bus Line
+	8130 970  8130 5620
+Wire Bus Line
+	7180 1260 7180 3470
+Wire Bus Line
+	3650 1260 3650 3470
+Wire Bus Line
+	14650 970  14650 5820
+Wire Bus Line
+	11550 970  11550 5620
 $EndSCHEMATC
